File: midi base/midi base.kicad_sch (KiCad schematic)
At the start: 56 parts, among them J1 USB_B, J10 AudioJack2, J2 USB_B, J3 USB_C_Receptacle_PowerOnly_6P, J4 USB to Pi, J5 Pi Zero 2 W, J6 RJ45, J7 MIDI Out, J8 AudioJack2, J9 MIDI In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

Commit message: added models
Parts:
- J1: footprint Connector_USB:USB_B_Lumberg_2411_02_Horizontal -> Connector_USB:USB_B_OST_USB-B1HSxx_Horizontal
- J7, J9: footprint Connector_RJ:RJ12_Amphenol_54601-x06_Horizontal -> Connector_JST:JST_XH_B5B-XH-A_1x05_P2.50mm_Vertical
Connections:
- net GND: now also SW10.3, SW10.5
Changed lines of the file:
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@@
 	)
 	(junction
+		(at 373.38 19.05)
+		(diameter 0)
+		(color 0 0 0 0)
+	)
+	(junction
 		(at 358.14 19.05)
 		(diameter 0)
@@
 	)
 	(junction
+		(at 364.49 19.05)
+		(diameter 0)
+		(color 0 0 0 0)
+	)
+	(junction
 		(at 48.26 39.37)
 		(diameter 0)
@@
 	(wire
 		(pts
+			(xy 364.49 19.05) (xy 373.38 19.05)
+		)
+		(stroke
+			(width 0)
+			(type default)
+		)
+	)
+	(wire
+		(pts
 			(xy 314.96 184.15) (xy 314.96 176.53)
 		)
@@
 			)
 		)
-		(property "Footprint" "Connector_RJ:RJ12_Amphenol_54601-x06_Horizontal"
+		(property "Footprint" "Connector_JST:JST_XH_B5B-XH-A_1x05_P2.50mm_Vertical"
 			(at 327.66 195.58 0)
 			(effects
@@
 			)
 		)
-		(property "Footprint" "Connector_RJ:RJ12_Amphenol_54601-x06_Horizontal"
+		(property "Footprint" "Connector_JST:JST_XH_B5B-XH-A_1x05_P2.50mm_Vertical"
 			(at 306.07 195.58 0)
 			(effects
@@
 			)
 		)
-		(property "Footprint" "Connector_USB:USB_B_Lumberg_2411_02_Horizontal"
+		(property "Footprint" "Connector_USB:USB_B_OST_USB-B1HSxx_Horizontal"
 			(at 31.75 205.74 0)
 			(effects

Commit message: did some stuff
Parts:
- J6: footprint Connector_RJ:RJ45_Amphenol_54602-x08_Horizontal -> (none)
Connections:
- net +3.3V: now also J6.7, J6.8; no longer J6.1, J6.2
- net at R7.1: now also J6.3; no longer J6.6
- net at R8.1, U5.7 (B): now also J6.6; no longer J6.3
- no-connect marks 47 -> 48
Other:
- moved on the sheet: R8, R9

Commit message: started pcb layout
Parts:
- removed J10, J8: AudioJack2, Connector_Audio:Jack_speakON-6.35mm_Neutrik_NLJ2MDXX-H_Horizontal, symbol Connector_Audio:AudioJack2
- added H1, H2, H3, H4, H5, H6: MountingHole, MountingHole:MountingHole_3.2mm_M3, symbol Mechanical:MountingHole
- added J11: TS In, Connector_JST:JST_XH_B4B-XH-A_1x04_P2.50mm_Vertical, symbol Connector:Conn_01x04_Socket
- J6: footprint (none) -> Connector_RJ:RJ45_Amphenol_RJHSE5380
Connections:
- net GND: now also J11.2 (Pin_2), J11.4 (Pin_4)
- net at U6.16 (GPIO1): now also J11.1 (Pin_1)
- net at U6.15 (GPIO0): now also J11.3 (Pin_3)
Other:
- note added: "Mechanical"
- moved on the sheet: C1, C2, C3, C4, C5, C6, D1, D2, D3, D4, J1, J2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

Commit message: more pcb stuff
Parts:
- C4: footprint Capacitor_SMD:C_0402_1005Metric -> Capacitor_SMD:C_0603_1608Metric
Connections:
- net +3.3V: no longer J6.7, J6.8
- net +5V: now also J6.7, J6.8
Changed lines of the file:
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@@
 			)
 		)
-		(property "Footprint" "Capacitor_SMD:C_0402_1005Metric"
+		(property "Footprint" "Capacitor_SMD:C_0603_1608Metric"
 			(at 192.7352 99.06 0)
 			(effects
@@
 	(symbol
 		(lib_id "power:+3.3V")
-		(at 20.32 29.21 0)
-		(mirror y)
-		(unit 1)
-		(exclude_from_sim no)
-		(in_bom yes)
-		(on_board yes)
-		(dnp no)
-		(property "Reference" "#PWR029"
-			(at 20.32 33.02 0)
-			(effects
-				(font
-					(size 1.27 1.27)
-				)
-				(hide yes)
-			)
-		)
-		(property "Value" "+3.3V"
-			(at 20.32 25.4 0)
-			(effects
-				(font
-					(size 1.27 1.27)
-				)
-			)
-		)
-		(property "Footprint" ""
-			(at 20.32 29.21 0)
-			(effects
-				(font
-					(size 1.27 1.27)
-				)
-				(hide yes)
-			)
-		)
-		(property "Datasheet" ""
-			(at 20.32 29.21 0)
-			(effects
-				(font
-					(size 1.27 1.27)
-				)
-				(hide yes)
-			)
-		)
-		(property "Description" "Power symbol creates a global label with name \"+3.3V\""
-			(at 20.32 29.21 0)
-			(effects
-				(font
-					(size 1.27 1.27)
-				)
-				(hide yes)
-			)
-		)
-		(pin "1"
-		)
-		(instances
-			(project "midi base"
-				(path "/e729c3f8-cc13-410c-ad9b-73759ef91302"
-					(reference "#PWR029")
-					(unit 1)
-				)
-			)
-		)
-	)
-	(symbol
-		(lib_id "power:+3.3V")
 		(at 156.21 107.95 90)
 		(unit 1)
@@
 					(unit 1)
 				)
+			)
+		)
+	)
+	(symbol
+		(lib_id "power:+5V")
+		(at 20.32 29.21 0)
+		(unit 1)
+		(exclude_from_sim no)
+		(in_bom yes)
+		(on_board yes)
+		(dnp no)
+		(fields_autoplaced yes)
+		(property "Reference" "#PWR029"
+			(at 20.32 33.02 0)
+			(effects
+				(font
+					(size 1.27 1.27)
+				)
+				(hide yes)
+			)
+		)
+		(property "Value" "+5V"
+			(at 20.32 24.13 0)
+			(effects
+				(font
+					(size 1.27 1.27)
+				)
+			)
+		)
+		(property "Footprint" ""
+			(at 20.32 29.21 0)
+			(effects
+				(font
+					(size 1.27 1.27)
+				)
+				(hide yes)
+			)
+		)
+		(property "Datasheet" ""
+			(at 20.32 29.21 0)
+			(effects
+				(font
+					(size 1.27 1.27)
+				)
+				(hide yes)
+			)
+		)
+		(property "Description" "Power symbol creates a global label with name \"+5V\""
+			(at 20.32 29.21 0)
+			(effects
+				(font
+					(size 1.27 1.27)
+				)
+				(hide yes)
+			)
+		)
+		(pin "1"
+		)
+		(instances
+			(project "midi base"
+				(path "/e729c3f8-cc13-410c-ad9b-73759ef91302"
+					(reference "#PWR029")
+					(unit 1)
+				)
