File: midi base/midi base.kicad_pcb (KiCad board)
At the start: 2 copper layers, 56 parts, among them J1 USB_B, J10 AudioJack2, J2 USB_B, J3 USB_C_Receptacle_PowerOnly_6P, J4 USB to Pi, J5 Pi Zero 2 W, J6 RJ45, J7 MIDI Out, J8 AudioJack2, J9 MIDI In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

Commit message: added models
Parts:
- J1: footprint Connector_USB:USB_B_Lumberg_2411_02_Horizontal -> Connector_USB:USB_B_OST_USB-B1HSxx_Horizontal
- J7, J9: footprint Connector_RJ:RJ12_Amphenol_54601-x06_Horizontal -> Connector_JST:JST_XH_B5B-XH-A_1x05_P2.50mm_Vertical
- moved J9 14.3 mm to (92.8, 123.7)
- moved J10 3.13 mm to (152.2, 120.5)
- moved J7 2.15 mm to (88.0, 115.8)

Commit message: did some stuff
Parts:
- removed J6: RJ45, Connector_RJ:RJ45_Amphenol_54602-x08_Horizontal
- added J11: RJ45_LED_Shielded, Connector_RJ:RJ45_Abracon_ARJP11A-MA_Horizontal, F.Cu at (176.4, 33.9)
- moved U2 6.37 mm to (198.8, 43.5)
Connections:
- SW10 pad 3: Net-(SW10-Pad3) -> GND
- SW10 pad 5: Net-(SW10-Pad3) -> GND

Commit message: started pcb layout
Parts:
- removed J10, J8: AudioJack2, Connector_Audio:Jack_speakON-6.35mm_Neutrik_NLJ2MDXX-H_Horizontal
- added H1: MountingHole, MountingHole:MountingHole_3.2mm_M3, F.Cu at (77.5, 59.1)
- added H2: MountingHole, MountingHole:MountingHole_3.2mm_M3, F.Cu at (219.7, 59.1)
- added H3: MountingHole, MountingHole:MountingHole_3.2mm_M3, F.Cu at (77.5, 150.5)
- added H4: MountingHole, MountingHole:MountingHole_3.2mm_M3, F.Cu at (219.7, 150.5)
- added H5: MountingHole, MountingHole:MountingHole_3.2mm_M3, F.Cu at (148.6, 59.1)
- added H6: MountingHole, MountingHole:MountingHole_3.2mm_M3, F.Cu at (148.6, 150.5)
- added J6: RJ45, Connector_RJ:RJ45_Amphenol_RJHSE5380, F.Cu at (-16.4, 50.2)
- J11: value RJ45_LED_Shielded -> TS In; footprint Connector_RJ:RJ45_Abracon_ARJP11A-MA_Horizontal -> Connector_JST:JST_XH_B4B-XH-A_1x04_P2.50mm_Vertical
- moved J11 211.0 mm to (-24.2, 99.3)
- moved J9 201.1 mm to (-108.2, 130.3)
- moved J1 195.8 mm to (-41.1, 50.3)
- moved J2 195.8 mm to (-41.1, 68.3)
- moved J3 195.8 mm to (-91.2, 141.5)
- moved J4 195.8 mm to (-109.3, 140.2)
- moved J7 195.8 mm to (-107.8, 121.1)
- moved SW1 195.8 mm to (-79.8, 121.9)
- moved SW2 195.8 mm to (-79.8, 137.1)
- moved U2 195.8 mm to (3.09, 48.8)
- moved D1 195.8 mm to (-1.23, 63.6)
- moved D2 195.8 mm to (-1.23, 66.2)
- moved D3 195.8 mm to (-1.23, 68.7)
- moved D4 195.8 mm to (-1.23, 71.3)
- moved R18 195.8 mm to (-4.72, 67.2)
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Connections:
- J11 pad 1: +3.3V -> Net-(J11-Pin_1)
- J11 pad 2: +3.3V -> GND
- J11 pad 3: Net-(U5-B) -> Net-(J11-Pin_3)
- R7 pad 1: Net-(J11-Pad6) -> Net-(J6-Pad3)
- U6 pad 15: Net-(U6-GPIO0) -> Net-(J11-Pin_3)
- U6 pad 16: Net-(U6-GPIO1) -> Net-(J11-Pin_1)
Routing:
- net Net-(U4-GPA6): track 0.00 -> 51.9 mm, vias 0 -> 2
- net Net-(U4-GPA1): track 0.00 -> 48.8 mm
- net Net-(U4-GPA4): track 0.00 -> 39.5 mm
- net Net-(U4-GPA3): track 0.00 -> 30.6 mm
- net Net-(U4-GPA7): track 0.00 -> 15.2 mm, vias 0 -> 2
- net +3.3V: track 0.00 -> 11.4 mm
- net Net-(R10-Pad2): track 0.00 -> 9.65 mm
- net Net-(U4-~{RESET}): track 0.00 -> 9.48 mm
- net Net-(U4-GPA5): track 0.00 -> 8.89 mm
- net GND: track 0.00 -> 1.73 mm, vias 0 -> 4
- added copper zone on B.Cu, net GND
- added copper zone on F.Cu, net GND
Other:
- board outline added: 152.4 x 101.6 mm

Commit message: more pcb updaytes
Routing:
- net Net-(U4-GPA0): track 0.00 -> 85.6 mm, vias 0 -> 2
- net Net-(U4-GPA2): track 0.00 -> 66.0 mm, vias 0 -> 2
- net Net-(R12-Pad2): track 0.00 -> 9.65 mm
- net Net-(R16-Pad2): track 0.00 -> 9.52 mm
- net Net-(R14-Pad2): track 0.00 -> 9.52 mm
- net Net-(R11-Pad2): track 0.00 -> 6.99 mm
- net Net-(R17-Pad2): track 0.00 -> 6.98 mm
- net Net-(R15-Pad2): track 0.00 -> 6.98 mm
- net Net-(R13-Pad2): track 0.00 -> 6.98 mm
- net Net-(U4-GPA4): track 39.5 -> 40.6 mm
- net Net-(U4-GPA1): track 48.8 -> 49.4 mm, vias 0 -> 2

Commit message: more pcb stuff
Parts:
- C4: footprint Capacitor_SMD:C_0402_1005Metric -> Capacitor_SMD:C_0603_1608Metric
- moved J3 311.6 mm to (208.9, 57.8), turned to 180 degrees
- moved J4 292.5 mm to (178.3, 86.9), turned to 180 degrees
- moved SW1 287.9 mm to (206.3, 153.7), turned to 90 degrees
- moved J9 277.7 mm to (168.3, 104.1)
- moved J7 277.3 mm to (168.3, 95.2)
- moved SW2 271.9 mm to (191.6, 153.7), turned to 90 degrees
- moved R1 267.1 mm to (210.1, 63.6), turned to -90 degrees
- moved R2 265.9 mm to (208.3, 63.6), turned to -90 degrees
- moved C1 262.3 mm to (205.6, 62.9), turned to 180 degrees
- moved U3 260.4 mm to (205.6, 66.6), turned to -90 degrees
- moved Y1 237.6 mm to (179.4, 71.1)
- moved J1 233.5 mm to (191.8, 66.9), turned to 90 degrees
- moved C2 232.5 mm to (180.1, 69.6)
- moved C3 231.0 mm to (178.0, 69.6), turned to 180 degrees
- moved U6 217.1 mm to (159.0, 97.0)
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Connections:
- J6 pad 7: +3.3V -> +5V
- J6 pad 8: +3.3V -> +5V
Routing:
- net +5V: track 0.00 -> 349.1 mm, vias 0 -> 10
- net GPIO_14: track 0.00 -> 127.8 mm, vias 0 -> 2
- net GPIO_15: track 0.00 -> 124.6 mm, vias 0 -> 4
- net GPIO_4: track 0.00 -> 124.3 mm, vias 0 -> 2
- net GPIO_26: track 0.00 -> 123.7 mm, vias 0 -> 6
- net GPIO_12: track 0.00 -> 103.5 mm, vias 0 -> 2
- net Net-(U4-GPB0): track 0.00 -> 75.6 mm, vias 0 -> 2
- net Net-(U4-GPB1): track 0.00 -> 64.6 mm, vias 0 -> 2
- net Net-(U4-GPB2): track 0.00 -> 62.1 mm, vias 0 -> 2
- net Net-(U4-GPB4): track 0.00 -> 59.1 mm, vias 0 -> 2
- net Net-(U4-GPB3): track 0.00 -> 49.0 mm, vias 0 -> 4
- net Net-(U4-GPB6): track 0.00 -> 44.5 mm, vias 0 -> 2
- net Net-(U4-GPB5): track 0.00 -> 42.8 mm, vias 0 -> 2
- net +3.3V: track 11.4 -> 48.0 mm
- net Net-(J1-D+): track 0.00 -> 33.0 mm, vias 0 -> 2
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- added copper zone on F.Cu, net +3.3V
- added copper zone on B.Cu, net +5V
- added copper zone on F.Cu, net +5V

Commit message: even more pcb things
Routing:
- net GPIO_2: track 31.0 -> 65.1 mm, vias 2 -> 4
Changed lines of the file:
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@@
+	)
+	(segment
+		(start 161.8665 101.5415)
+		(end 161.8665 100.603)
+		(width 0.2)
+		(layer "F.Cu")
+		(net 51)
 	)
 	(segment
@@
 		(end 138.684 147.32)
 		(width 0.3)
+		(layer "F.Cu")
+		(net 51)
+	)
+	(segment
+		(start 148.59 125.975001)
+		(end 150.504605 124.060396)
+		(width 0.2)
 		(layer "F.Cu")
 		(net 51)
@@
 	)
 	(segment
+		(start 161.925 101.6)
+		(end 161.8665 101.5415)
+		(width 0.2)
+		(layer "F.Cu")
+		(net 51)
+	)
+	(segment
+		(start 161.29 104.14)
+		(end 161.925 103.505)
+		(width 0.2)
+		(layer "F.Cu")
+		(net 51)
+	)
+	(segment
+		(start 151.529604 124.060396)
+		(end 158.75 116.84)
+		(width 0.2)
+		(layer "F.Cu")
+		(net 51)
+	)
+	(segment
+		(start 160.67 104.14)
+		(end 161.29 104.14)
+		(width 0.2)
+		(layer "F.Cu")
+		(net 51)
+	)
+	(segment
+		(start 150.504605 124.060396)
+		(end 151.529604 124.060396)
+		(width 0.2)
+		(layer "F.Cu")
+		(net 51)
+	)
+	(segment
 		(start 138.43 149.86)
 		(end 138.43 147.574)
 		(width 0.3)
 		(layer "F.Cu")
+		(net 51)
+	)
+	(segment
+		(start 148.59 127)
+		(end 148.59 125.975001)
+		(width 0.2)
+		(layer "F.Cu")
+		(net 51)
+	)
+	(segment
+		(start 158.75 116.84)
+		(end 158.75 104.14)
+		(width 0.2)
+		(layer "F.Cu")
+		(net 51)
+	)
+	(segment
+		(start 161.925 103.505)
+		(end 161.925 101.6)
+		(width 0.2)
+		(layer "F.Cu")
+		(net 51)
+	)
+	(via
+		(at 160.67 104.14)
+		(size 0.6)
+		(drill 0.3)
+		(layers "F.Cu" "B.Cu")
 		(net 51)
 	)
@@
 		(net 51)
 	)
+	(via
+		(at 158.75 104.14)
+		(size 0.6)
+		(drill 0.3)
+		(layers "F.Cu" "B.Cu")
+		(net 51)
+	)
 	(segment
 		(start 138.684 147.32)
@@
 		(layer "B.Cu")
 		(net 51)
+	)
+	(segment
+		(start 158.75 104.14)
+		(end 160.67 104.14)
+		(width 0.2)
+		(layer "B.Cu")
+		(net 51)

Commit message: did some funky file stuff
Parts:
- moved R7 3.63 mm to (88.1, 75.1), turned to -90 degrees
- moved R18 1.03 mm to (163.4, 100.6), turned to 90 degrees
- moved R5 0.72 mm to (173.9, 79.8), turned to 180 degrees
- moved R4 0.72 mm to (178.3, 79.8), turned to 0 degrees
- moved J3 0.38 mm to (208.9, 57.4)
Routing:
- net +3.3V: track 48.0 -> 359.1 mm, vias 0 -> 2
- net GPIO_19: track 0.00 -> 134.2 mm, vias 0 -> 6
- net GPIO_13: track 0.00 -> 125.3 mm, vias 0 -> 6
- net GPIO_9: track 0.00 -> 119.3 mm, vias 0 -> 4
- net GPIO_11: track 0.00 -> 116.4 mm, vias 0 -> 6
- net GPIO_10: track 0.00 -> 107.4 mm, vias 0 -> 4
- net GPIO_20: track 0.00 -> 105.2 mm, vias 0 -> 2
- net GPIO_25: track 0.00 -> 104.8 mm, vias 0 -> 6
- net GPIO_8: track 0.00 -> 102.9 mm, vias 0 -> 5
- net GPIO_23: track 0.00 -> 100.8 mm, vias 0 -> 4
- net GPIO_16: track 0.00 -> 94.3 mm
- net GPIO_24: track 1.76 -> 87.5 mm, vias 0 -> 8
- net GPIO_3: track 31.6 -> 66.7 mm
- net Net-(U6-RX): track 0.00 -> 29.6 mm, vias 0 -> 2
- net Net-(U6-TX): track 0.00 -> 24.3 mm, vias 0 -> 2
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